Commit message: Add tags to Innopoils duckietown map

File: catkin_ws/src/30-localization-and-planning/duckietown_description/urdf/innopolis.urdf.xacro (robot description, xacro)
@@ -4,12 +4,12 @@
         <!--Parameters-->
         <xacro:property name="tile_width" value="0.595"/>
-        <xacro:property name="pos_0" value="0.09 0.035"/>
-        <xacro:property name="pos_1" value="0.035 0.09"/>
-        <xacro:property name="pos_2" value="-0.035 0.09"/>
-        <xacro:property name="pos_3" value="-0.09 0.035"/>
-        <xacro:property name="pos_4" value="-0.09 -0.035"/>
-        <xacro:property name="pos_5" value="-0.035 -0.09"/>
-        <xacro:property name="pos_6" value="0.035 -0.09"/>
-        <xacro:property name="pos_7" value="0.09 -0.035"/>
+        <xacro:property name="pos_0" value="0.05 0.03"/>
+        <xacro:property name="pos_1" value="0.03 0.05"/>
+        <xacro:property name="pos_2" value="-0.03 0.05"/>
+        <xacro:property name="pos_3" value="-0.05 0.03"/>
+        <xacro:property name="pos_4" value="-0.05 -0.03"/>
+        <xacro:property name="pos_5" value="-0.03 -0.05"/>
+        <xacro:property name="pos_6" value="0.03 -0.05"/>
+        <xacro:property name="pos_7" value="0.05 -0.03"/>
         <!--Include the tile and tag macros-->
         <xacro:include filename="$(find duckietown_description)/urdf/macros.urdf.xacro"/>
@@ -55,3 +55,6 @@
         <xacro:tile visible="false" x="5" y="4"/>
         <!--Describe the tags-->
+        <xacro:tag id="66" pos="${pos_0}" rotation="180" x="5" y="2"/>
+        <xacro:tag id="62" pos="${pos_5}" rotation="270" x="5" y="3"/>
+        <xacro:tag id="58" pos="${pos_7}" rotation="90" x="4" y="2"/>
     </robot>
