Commit message: Add stoplines to urdf

File: catkin_ws/src/30-localization-and-planning/duckietown_description/urdf/macros.urdf.xacro (robot description, xacro)
@@ -1,22 +1,60 @@
 <?xml version="1.0"?>
 <robot name="macros" xmlns:xacro="http://www.ros.org/wiki/xacro">
-    <xacro:property name="pi" value="3.14159265359" />
-    <xacro:property name="tile_thickness" value="0.01" />
+    <xacro:property name="pi" value="3.14159265359"/>
+    <xacro:property name="tile_thickness" value="0.01"/>
+    <xacro:property name="road_width" value="0.435"/>
+    <xacro:property name="stopline_offset" value="0"/>
     <!-- Defines a tile link and joint-->
     <xacro:macro name="tile" params="x y type:=empty rotation:=0 visible:=true">
         <link name="tile_${x}_${y}">
-            <xacro:if value="${visible}" >
+            <xacro:if value="${visible}">
                 <visual>
-                    <origin xyz="${tile_width/2} ${tile_width/2} ${-tile_thickness/2}" rpy="0 0 ${rotation * pi/180}"/>
+                    <origin xyz="0 0 ${-tile_thickness/2}"/>
                     <geometry>
-                        <mesh filename="package://duckietown_description/urdf/meshes/${type}.dae" />
+                        <mesh filename="package://duckietown_description/urdf/meshes/${type}.dae"/>
                     </geometry>
                 </visual>
             </xacro:if>
         </link>
+        <!-- Bottom stop-line -->
+        <xacro:if value="${type == '4way'}">
+            <link name="stopline_${x}_${y}_0"/>
+            <joint name="tile_${x}_${y}_to_stopline_0" type="fixed">
+                <parent link="tile_${x}_${y}"/>
+                <child link="stopline_${x}_${y}_0"/>
+                <origin xyz="${(road_width)/4} ${-tile_width/2 + stopline_offset} 0" rpy="0 0 ${pi/2}"/>
+            </joint>
+        </xacro:if>
+        <xacro:if value="${type == '3way' or type == '4way'}">
+            <link name="stopline_${x}_${y}_1"/>
+            <joint name="tile_${x}_${y}_to_stopline_1" type="fixed">
+                <parent link="tile_${x}_${y}"/>
+                <child link="stopline_${x}_${y}_1"/>
+                <origin xyz="${tile_width/2 - stopline_offset} ${(road_width)/4} 0" rpy="0 0 ${pi}"/>
+            </joint>
+            <link name="stopline_${x}_${y}_2"/>
+            <joint name="tile_${x}_${y}_to_stopline_2" type="fixed">
+                <parent link="tile_${x}_${y}"/>
+                <child link="stopline_${x}_${y}_2"/>
+                <origin xyz="${-(road_width)/4} ${tile_width/2 - stopline_offset} 0"  rpy="0 0 ${-pi/2}"/>
+            </joint>
+            <link name="stopline_${x}_${y}_3"/>
+            <joint name="tile_${x}_${y}_to_stopline_3" type="fixed">
+                <parent link="tile_${x}_${y}"/>
+                <child link="stopline_${x}_${y}_3"/>
+                <origin xyz="${-tile_width/2 + stopline_offset} ${-(road_width)/4} 0"/>
+            </joint>
+        </xacro:if>
         <joint name="world_to_tile_${x}_${y}" type="fixed">
-            <parent link="world" />
-            <child link="tile_${x}_${y}" />
-            <origin xyz="${tile_width * x} ${tile_width * y} 0" />
+            <parent link="world"/>
+            <child link="tile_${x}_${y}"/>
+            <origin xyz="${tile_width * x + tile_width / 2} ${tile_width * y + tile_width / 2} 0"
+                    rpy="0 0 ${rotation * pi/180}"/>
+        </joint>
+        <link name="cell_point_${x}_${y}"/>
+        <joint name="world_to_cell_point_${x}_${y}" type="fixed">
+            <parent link="world"/>
+            <child link="cell_point_${x}_${y}"/>
+            <origin xyz="${tile_width * x} ${tile_width * y} 0"/>
         </joint>
     </xacro:macro>
@@ -25,13 +63,13 @@
         <link name="tag_${id}">
             <visual>
-                <origin xyz="-0.0254 -0.0254 0" />
+                <origin xyz="-0.0254 -0.0254 0"/>
                 <geometry>
-                    <mesh filename="package://duckietown_description/urdf/meshes/tags/tag_${id}.dae" />
+                    <mesh scale="0.005 0.005 0.005" filename="package://duckietown_description/urdf/meshes/tags/tag_${id}.dae"/>
                 </geometry>
             </visual>
         </link>
         <joint name="world_to_tag_${id}" type="fixed">
-            <parent link="tile_${x}_${y}" />
-            <child link="tag_${id}" />
+            <parent link="cell_point_${x}_${y}"/>
+            <child link="tag_${id}"/>
             <origin xyz="${pos} 0" rpy="0 0 ${rotation * pi/180}"/>
         </joint>
